File: RGBMatrix.kicad_sch (KiCad schematic)
At the start: 273 parts, among them U1 74LS596, U10 FDG6323L-TP, U11 FDG6323L-TP, U12 FDG6323L-TP, U13 FDG6323L-TP, U14 FDG6323L-TP, U15 FDG6323L-TP, U16 FDG6323L-TP, U17 FDG6323L-TP, U18 FDG6323L-TP, U19 FDG6323L-TP, U2 74LS596, U20 FDG6323L-TP, U21 FDG6323L-TP, U22 FDG6323L-TP, U23 FDG6323L-TP, U24 FDG6323L-TP, U3 74LS596, U4 74LS596, U5 74LS596, U6 74LS596, U7 FDG6323L-TP, U8 74LS596, U9 74LS596

Commit message: refactoring
Refactoring the whole fucking design.
Parts:
- removed C10, C11, C12, C13, C14, C15, C16, C17, C18, C19, C20, C6, C7, C8, C9: C, Capacitor_SMD:C_0402_1005Metric, symbol Device:C
- removed RN11, RN13: 0Ohm, Resistor_SMD:R_Array_Convex_8x0602, symbol Device:R_Pack08
- added J1, J2, J3, J4: Conn_01x07, Connector_PinSocket_2.54mm:PinSocket_1x07_P2.54mm_Vertical, symbol Connector_Generic:Conn_01x07
- added J5: Conn_01x08, Connector_PinSocket_2.54mm:PinSocket_1x08_P2.54mm_Vertical, symbol Connector_Generic:Conn_01x08
- C1, C2, C29, C30: footprint Capacitor_SMD:C_0805_2012Metric -> Capacitor_SMD:C_0603_1608Metric
Connections:
- net +3.3V: now also C5.1, J1.2 (Pin_2), J2.2 (Pin_2), J3.6 (Pin_6), J5.6 (Pin_6)
- net A16: no longer C5.1
- net A_IN: now also J3.4 (Pin_4), J5.5 (Pin_5)
- net B01: now also RN4.15 (R2.2); no longer RN3.9 (R8.2)
- net B02: now also RN4.14 (R3.2); no longer RN3.10 (R7.2)
- net B03: now also RN4.13 (R4.2); no longer RN3.11 (R6.2)
- net B04: now also RN4.12 (R5.2); no longer RN3.12 (R5.2)
- net B05: now also RN4.11 (R6.2); no longer RN3.13 (R4.2)
- net B06: now also RN4.10 (R7.2); no longer RN3.14 (R3.2)
- net B08: now also RN3.14 (R3.2); no longer RN4.10 (R7.2)
- net B09: now also RN3.13 (R4.2); no longer RN4.11 (R6.2)
- net B10: now also RN3.12 (R5.2); no longer RN4.12 (R5.2)
- net B11: now also RN3.11 (R6.2); no longer RN4.13 (R4.2)
- net B12: now also RN3.10 (R7.2); no longer RN4.14 (R3.2)
- net B13: now also RN3.9 (R8.2); no longer RN4.15 (R2.2)
- net B_IN: now also U4.14 (SER), J1.3 (Pin_3), J4.6 (Pin_6); no longer U3.14 (SER)
- net COL01: now also RN8.10 (R7.2); no longer RN8.16 (R1.2)
- net COL02: now also RN8.11 (R6.2); no longer RN8.15 (R2.2)
- net COL03: now also RN8.12 (R5.2); no longer RN8.14 (R3.2)
- net COL05: now also RN8.14 (R3.2); no longer RN8.12 (R5.2)
- net COL06: now also RN8.15 (R2.2); no longer RN8.11 (R6.2)
- net COL07: now also RN8.16 (R1.2); no longer RN8.10 (R7.2)
- net COL09: now also RN7.10 (R7.2); no longer RN7.16 (R1.2)
- net COL10: now also RN7.11 (R6.2); no longer RN7.15 (R2.2)
- net COL11: now also RN7.12 (R5.2); no longer RN7.14 (R3.2)
- net COL13: now also RN7.14 (R3.2); no longer RN7.12 (R5.2)
- net COL14: now also RN7.15 (R2.2); no longer RN7.11 (R6.2)
- net COL15: now also RN7.16 (R1.2); no longer RN7.10 (R7.2)
- net G01: now also RN6.15 (R2.2); no longer RN5.9 (R8.2)
- net G02: now also RN6.14 (R3.2); no longer RN5.10 (R7.2)
- net G03: now also RN6.13 (R4.2); no longer RN5.11 (R6.2)
- net G04: now also RN6.12 (R5.2); no longer RN5.12 (R5.2)
- net G05: now also RN6.11 (R6.2); no longer RN5.13 (R4.2)
- net G06: now also RN6.10 (R7.2); no longer RN5.14 (R3.2)
- net G08: now also RN5.14 (R3.2); no longer RN6.10 (R7.2)
- net G09: now also RN5.13 (R4.2); no longer RN6.11 (R6.2)
- net G10: now also RN5.12 (R5.2); no longer RN6.12 (R5.2)
- net G11: now also RN5.11 (R6.2); no longer RN6.13 (R4.2)
- net G12: now also RN5.10 (R7.2); no longer RN6.14 (R3.2)
- net G13: now also RN5.9 (R8.2); no longer RN6.15 (R2.2)
- net GND: now also U10.1 (R2), U11.1 (R2), U12.1 (R2), U13.1 (R2), U14.1 (R2), U15.1 (R2), U16.1 (R2), U17.1 (R2), U18.1 (R2), U19.1 (R2), U20.1 (R2), U21.1 (R2), U22.1 (R2), U23.1 (R2), U24.1 (R2), U7.1 (R2), J1.1 (Pin_1), J2.1 (Pin_1), J3.7 (Pin_7), J4.7 (Pin_7), J5.7 (Pin_7)
- net G_IN: now also U6.14 (SER), J1.4 (Pin_4), J4.5 (Pin_5); no longer U5.14 (SER)
- net R01: now also RN1.9 (R8.2); no longer RN1.15 (R2.2)
- net R02: now also RN1.10 (R7.2); no longer RN1.14 (R3.2)
- net R03: now also RN1.11 (R6.2); no longer RN1.13 (R4.2)
- net R05: now also RN1.13 (R4.2); no longer RN1.11 (R6.2)
- net R06: now also RN1.14 (R3.2); no longer RN1.10 (R7.2)
- net R07: now also RN1.15 (R2.2); no longer RN1.9 (R8.2)
- net R08: now also RN2.10 (R7.2); no longer RN2.15 (R2.2)
- net R09: now also RN2.11 (R6.2); no longer RN2.14 (R3.2)
- net R10: now also RN2.12 (R5.2); no longer RN2.13 (R4.2)
- net R11: now also RN2.13 (R4.2); no longer RN2.12 (R5.2)
- net R12: now also RN2.14 (R3.2); no longer RN2.11 (R6.2)
- net R13: now also RN2.15 (R2.2); no longer RN2.10 (R7.2)
- net RCLK_A: now also J3.3 (Pin_3), J5.3 (Pin_3)
- net RCLK_RGB: now also J1.5 (Pin_5), J2.5 (Pin_5), J4.3 (Pin_3)
- net R_IN: now also J2.4 (Pin_4), J4.4 (Pin_4)
- net SRCLK_A: now also J3.2 (Pin_2), J5.2 (Pin_2)
- net SRCLK_RGB: now also J1.6 (Pin_6), J2.6 (Pin_6), J4.2 (Pin_2)
- net V_LED: now also J3.5 (Pin_5), J5.8 (Pin_8)
- net _SRCLR_A: now also J3.1 (Pin_1), J5.1 (Pin_1)
- net _SRCLR_RGB: now also J1.7 (Pin_7), J2.7 (Pin_7), J4.1 (Pin_1)
- net at U7.6 (R1C1): now also RN10.11 (R6.2); no longer RN12.10 (R7.2)
- net at RN5.2 (R2.1): now also U5.1 (QB); no longer U5.7 (QH)
- net at RN5.3 (R3.1): now also U5.2 (QC); no longer U5.6 (QG)
- net at RN5.4 (R4.1): now also U5.3 (QD); no longer U5.5 (QF)
- net at RN5.6 (R6.1): now also U5.5 (QF); no longer U5.3 (QD)
- net at RN5.7 (R7.1): now also U5.6 (QG); no longer U5.2 (QC)
- net at RN5.8 (R8.1): now also U5.7 (QH); no longer U5.1 (QB)
- net at U5.9 (QH'): no longer U6.14 (SER)
- net at U9.1 (QB): now also RN8.1 (R1.1); no longer RN8.7 (R7.1)
- net at U9.2 (QC): now also RN8.2 (R2.1); no longer RN8.6 (R6.1)
- net at U9.3 (QD): now also RN8.3 (R3.1); no longer RN8.5 (R5.1)
- net at U9.5 (QF): now also RN8.5 (R5.1); no longer RN8.3 (R3.1)
- net at U9.6 (QG): now also RN8.6 (R6.1); no longer RN8.2 (R2.1)
- net at U9.7 (QH): now also RN8.7 (R7.1); no longer RN8.1 (R1.1)
- net at U24.6 (R1C1): now also RN12.15 (R2.2); no longer RN12.12 (R5.2)
- net at U10.6 (R1C1): now also RN10.12 (R5.2); no longer RN12.14 (R3.2)
- net at U3.9 (QH'): no longer U4.14 (SER)
- net at U4.2 (QC): now also RN4.2 (R2.1); no longer RN4.7 (R7.1)
- net at U4.3 (QD): now also RN4.3 (R3.1); no longer RN4.6 (R6.1)
- net at U4.4 (QE): now also RN4.4 (R4.1); no longer RN4.5 (R5.1)
- net at U4.5 (QF): now also RN4.5 (R5.1); no longer RN4.4 (R4.1)
- net at U4.6 (QG): now also RN4.6 (R6.1); no longer RN4.3 (R3.1)
- net at U4.7 (QH): now also RN4.7 (R7.1); no longer RN4.2 (R2.1)
- net at U4.9 (QH'): now also U3.14 (SER)
- net at RN10.10 (R7.2): now also U14.6 (R1C1); no longer U11.6 (R1C1)
- net at U18.6 (R1C1): now also RN12.11 (R6.2); no longer RN10.11 (R6.2)
- net at U22.6 (R1C1): now also RN12.12 (R5.2); no longer RN10.12 (R5.2)
- net at RN10.13 (R4.2): now also U11.6 (R1C1); no longer U16.6 (R1C1)
- net at RN10.14 (R3.2): now also U15.6 (R1C1); no longer U12.6 (R1C1)
- net at RN10.15 (R2.2): now also U12.6 (R1C1); no longer U17.6 (R1C1)
- net at RN10.16 (R1.2): now also U16.6 (R1C1); no longer U21.6 (R1C1)
- net at RN10.9 (R8.2): now also U13.6 (R1C1); no longer U15.6 (R1C1)
- net at RN12.9 (R8.2): now also U21.6 (R1C1); no longer U13.6 (R1C1)
- net at RN3.2 (R2.1): now also U3.1 (QB); no longer U3.7 (QH)
- net at RN3.3 (R3.1): now also U3.2 (QC); no longer U3.6 (QG)
- net at RN3.4 (R4.1): now also U3.3 (QD); no longer U3.5 (QF)
- net at RN3.6 (R6.1): now also U3.5 (QF); no longer U3.3 (QD)
- net at RN3.7 (R7.1): now also U3.6 (QG); no longer U3.2 (QC)
- net at RN3.8 (R8.1): now also U3.7 (QH); no longer U3.1 (QB)
- net at RN6.2 (R2.1): now also U6.2 (QC); no longer U6.7 (QH)
- net at RN6.3 (R3.1): now also U6.3 (QD); no longer U6.6 (QG)
- net at RN6.4 (R4.1): now also U6.4 (QE); no longer U6.5 (QF)
- net at RN6.5 (R5.1): now also U6.5 (QF); no longer U6.4 (QE)
- net at RN6.6 (R6.1): now also U6.6 (QG); no longer U6.3 (QD)
- net at RN6.7 (R7.1): now also U6.7 (QH); no longer U6.2 (QC)
- net at U20.6 (R1C1): now also RN12.14 (R3.2); no longer RN12.11 (R6.2)
- net at RN12.13 (R4.2): now also U19.6 (R1C1); no longer U14.6 (R1C1)
- net at RN1.2 (R2.1): now also U1.1 (QB); no longer U1.7 (QH)
- net at RN1.3 (R3.1): now also U1.2 (QC); no longer U1.6 (QG)
- net at RN1.4 (R4.1): now also U1.3 (QD); no longer U1.5 (QF)
- net at RN1.6 (R6.1): now also U1.5 (QF); no longer U1.3 (QD)
- net at RN1.7 (R7.1): now also U1.6 (QG); no longer U1.2 (QC)
- net at RN1.8 (R8.1): now also U1.7 (QH); no longer U1.1 (QB)
- net at U2.2 (QC): now also RN2.2 (R2.1); no longer RN2.7 (R7.1)
- net at U2.3 (QD): now also RN2.3 (R3.1); no longer RN2.6 (R6.1)
- net at U2.4 (QE): now also RN2.4 (R4.1); no longer RN2.5 (R5.1)
- net at U2.5 (QF): now also RN2.5 (R5.1); no longer RN2.4 (R4.1)
- net at U2.6 (QG): now also RN2.6 (R6.1); no longer RN2.3 (R3.1)
- net at U2.7 (QH): now also RN2.7 (R7.1); no longer RN2.2 (R2.1)
- net at U8.1 (QB): now also RN7.1 (R1.1); no longer RN7.7 (R7.1)
- net at U8.2 (QC): now also RN7.2 (R2.1); no longer RN7.6 (R6.1)
- net at U8.3 (QD): now also RN7.3 (R3.1); no longer RN7.5 (R5.1)
- net at U8.5 (QF): now also RN7.5 (R5.1); no longer RN7.3 (R3.1)
- net at U8.6 (QG): now also RN7.6 (R6.1); no longer RN7.2 (R2.1)
- net at U8.7 (QH): now also RN7.7 (R7.1); no longer RN7.1 (R1.1)
- net at U6.9 (QH'): now also U5.14 (SER)
- new net: RN12.10 (R7.2), U17.6 (R1C1)
- no-connect marks 30 -> 32
Other:
- moved on the sheet: RN1, RN10, RN12, RN3, RN4, RN5, RN6, RN7, RN8, U10, U11, U12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
