File: RGBMatrix.kicad_sch (KiCad schematic)
At the start: 261 parts, among them J1 Conn_01x07, J2 Conn_01x07, J3 Conn_01x07, J4 Conn_01x07, J5 Conn_01x08, U1 74LS596, U10 FDG6323L-TP, U11 FDG6323L-TP, U12 FDG6323L-TP, U13 FDG6323L-TP, U14 FDG6323L-TP, U15 FDG6323L-TP, U16 FDG6323L-TP, U17 FDG6323L-TP, U18 FDG6323L-TP, U19 FDG6323L-TP, U2 74LS596, U20 FDG6323L-TP, U21 FDG6323L-TP, U22 FDG6323L-TP, U23 FDG6323L-TP, U24 FDG6323L-TP, U3 74LS596, U4 74LS596, U5 74LS596, U6 74LS596, U7 FDG6323L-TP, U8 74LS596, U9 74LS596

Commit message: update
break down schemantic to panels, added controller and additional commponents, fixed
Parts:
- removed C1, C2, C29, C30: C, Capacitor_SMD:C_0603_1608Metric, symbol Device:C
- removed C21, C22, C23, C24, C25, C26, C27, C5: C, Capacitor_SMD:C_0402_1005Metric, symbol Device:C
- removed C3, C4: C, Capacitor_SMD:C_0805_2012Metric, symbol Device:C
- removed J1, J2, J3, J4: Conn_01x07, Connector_PinSocket_2.54mm:PinSocket_1x07_P2.54mm_Vertical, symbol Connector_Generic:Conn_01x07
- removed J5: Conn_01x08, Connector_PinSocket_2.54mm:PinSocket_1x08_P2.54mm_Vertical, symbol Connector_Generic:Conn_01x08
- removed LED1, LED10, LED100, LED101, LED102, LED103, LED104, LED105, LED106, LED107, LED108, LED109, LED11, LED110, LED111, LED112, LED113, LED114, LED115, LED116, LED117, LED118, LED119, LED12, LED120, LED121, LED122, LED123, LED124, LED125, LED126, LED127, LED128, LED129, LED13, LED130, LED131, LED132, LED133, LED134, LED135, LED136, LED137, LED138, LED139, LED14, LED140, LED141, LED142, LED143, LED144, LED145, LED146, LED147, LED148, LED149, LED15, LED150, LED151, LED152, LED153, LED154, LED155, LED156, LED157, LED158, LED159, LED16, LED160, LED161, LED162, LED163, LED164, LED165, LED166, LED167, LED168, LED169, LED17, LED170, LED171, LED172, LED173, LED174, LED175, LED176, LED177, LED178, LED179, LED18, LED180, LED181, LED182, LED183, LED184, LED185, LED186, LED187, LED188, LED189, LED19, LED190, LED191, LED192, LED193, LED194, LED195, LED196, LED197, LED198, LED199, LED2, LED20, LED200, LED201, LED202, LED203, LED204, LED205, LED206, LED207, LED208, LED21, LED22, LED23, LED24, LED25, LED26, LED27, LED28, LED29, LED3, LED30, LED31, LED32, LED33, LED34, LED35, LED36, LED37, LED38, LED39, LED4, LED40, LED41, LED42, LED43, LED44, LED45, LED46, LED47, LED48, LED49, LED5, LED50, LED51, LED52, LED53, LED54, LED55, LED56, LED57, LED58, LED59, LED6, LED60, LED61, LED62, LED63, LED64, LED65, LED66, LED67, LED68, LED69, LED7, LED70, LED71, LED72, LED73, LED74, LED75, LED76, LED77, LED78, LED79, LED8, LED80, LED81, LED82, LED83, LED84, LED85, LED86, LED87, LED88, LED89, LED9, LED90, LED91, LED92, LED93, LED94, LED95, LED96, LED97, LED98, LED99: UHD111A, LED:UHD111AFKAC3K23E1L3VG5ZB3Z3, symbol LED:UHD111A-FKA-C3K23E1L3VG5ZB3Z3
- removed RN1, RN2: 270Ohm, Resistor_SMD:R_Array_Convex_8x0602, symbol Device:R_Pack08
- removed RN10, RN12: 10kOhm, Resistor_SMD:R_Array_Convex_8x0602, symbol Device:R_Pack08
- removed RN3, RN4, RN5, RN6: 200Ohm, Resistor_SMD:R_Array_Convex_8x0602, symbol Device:R_Pack08
- removed RN7, RN8: 4.7kOhm, Resistor_SMD:R_Array_Convex_8x0602, symbol Device:R_Pack08
- removed U1, U2, U3, U4, U5, U6, U8, U9: 74LS596, Package_SO:TSSOP-16_4.4x5mm_P0.65mm, symbol 74xx:74LS596
- removed U10, U11, U12, U13, U14, U15, U16, U17, U18, U19, U20, U21, U22, U23, U24, U7: FDG6323L-TP, FDG6323L:FDG6323L, symbol FDG6323L:FDG6323L-TP
- added J5: USB_C_Receptacle_USB2.0_16P, Connector_USB:USB_C_Receptacle_HCTL_HC-TYPE-C-16P-01A, symbol Connector:USB_C_Receptacle_USB2.0_16P
- added R4, R8: 5.1k, Resistor_SMD:R_0603_1608Metric, symbol Device:R
- added U32: USBLC6-4SC6, Package_TO_SOT_SMD:SOT-23-6, symbol Power_Protection:USBLC6-4SC6
Connections:
- net GND: now also J5.A1 (GND), J5.A12 (GND), J5.B1 (GND), J5.B12 (GND), J5.SH (SHIELD), R4.2, R8.2, U32.2 (GND)
- new net: J5.B5 (CC2), R8.1
- new net: J5.A5 (CC1), R4.1
- new net +5V: J5.A4 (VBUS), J5.A9 (VBUS), J5.B4 (VBUS), J5.B9 (VBUS), U32.5 (VBUS)
- new net FrontPanel/D+: J5.A6 (D+), J5.B6 (D+), U32.3 (I/O2), U32.4 (I/O3)
- new net FrontPanel/D-: J5.A7 (D-), J5.B7 (D-), U32.1 (I/O1), U32.6 (I/O4)
- no-connect marks 32 -> 2
Other:
- added sheet FrontPanel (FrontPanel.kicad_sch)
- added sheet LedPanel (LedPanel.kicad_sch)
- added sheet LeftPanel (LeftPanel.kicad_sch)
- added sheet RightPanel (RightPanel.kicad_sch)
