File: RGBMatrixLeds.kicad_pcb (KiCad board)
At the start: 6 copper layers, 69 x 115 mm, 259 parts, among them J1 Conn_01x07, J2 Conn_01x07, J3 Conn_01x07, J4 Conn_01x07, J5 Conn_01x08, U1 74LS596, U10 FDG6323L-TP, U11 FDG6323L-TP, U12 FDG6323L-TP, U13 FDG6323L-TP, U14 FDG6323L-TP, U15 FDG6323L-TP, U16 FDG6323L-TP, U17 FDG6323L-TP, U18 FDG6323L-TP, U19 FDG6323L-TP, U2 74LS596, U20 FDG6323L-TP, U21 FDG6323L-TP, U22 FDG6323L-TP, U23 FDG6323L-TP, U24 FDG6323L-TP, U3 74LS596, U4 74LS596, U5 74LS596, U6 74LS596, U7 FDG6323L-TP, U8 74LS596, U9 74LS596

Commit message: refactoring
Refactoring the whole fucking design.
Parts:
- removed C22, C24, C25, C26, C27, C5: C, Capacitor_SMD:C_0402_1005Metric
- removed J1, J2, J3, J4: Conn_01x07, Connector_PinSocket_2.54mm:PinSocket_1x07_P2.54mm_Vertical
- removed J5: Conn_01x08, Connector_PinSocket_2.54mm:PinSocket_1x08_P2.54mm_Vertical
- removed RN1, RN2: 270Ohm, Resistor_SMD:R_Array_Convex_8x0602
- removed RN3, RN4, RN5, RN6: 200Ohm, Resistor_SMD:R_Array_Convex_8x0602
- removed U1, U2, U3, U4, U5, U6: 74LS596, Package_SO:TSSOP-16_4.4x5mm_P0.65mm
Routing:
- net RCLK_RGB: track 126.0 -> 0.00 mm, vias 8 -> 0
- net SRCLK_RGB: track 119.5 -> 0.00 mm, vias 8 -> 0
- net _SRCLR_RGB: track 114.5 -> 0.00 mm, vias 8 -> 0
- net +3.3V: track 127.7 -> 24.7 mm, vias 11 -> 3
- net R_IN: track 87.9 -> 0.00 mm, vias 2 -> 0
- net B_IN: track 78.7 -> 0.00 mm, vias 2 -> 0
- net G_IN: track 57.4 -> 0.00 mm, vias 2 -> 0
- net V_LED: track 128.6 -> 84.3 mm
- net G05: track 58.1 -> 20.9 mm, vias 18 -> 16
- net A_IN: track 58.6 -> 23.7 mm
- net G04: track 53.7 -> 20.9 mm, vias 18 -> 16
- net RCLK_A: track 59.1 -> 26.9 mm
- net SRCLK_A: track 58.1 -> 27.9 mm
- net G03: track 49.4 -> 20.9 mm, vias 18 -> 16
- net _SRCLR_A: track 54.9 -> 27.2 mm
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- removed copper zone on B.Cu, net +3.3V
Other:
- board size 69 x 115 mm -> 23.5 x 50 mm
- board text removed: "Kifér az"
- board text removed: "Lopják a"
- board text removed: "Mátrixot"
- board text removed: "Tedd vissza!"
- board text removed: "VESZ- TETTEM"
- board text removed: "You like looking at design files, don't you?"
- board text removed: "ablakon"
