File: LedPanel.kicad_sch (KiCad schematic)
At the start: 238 parts, among them U10 FDG6323L-TP, U11 FDG6323L-TP, U12 FDG6323L-TP, U13 FDG6323L-TP, U14 FDG6323L-TP, U15 FDG6323L-TP, U16 FDG6323L-TP, U17 FDG6323L-TP, U18 FDG6323L-TP, U19 FDG6323L-TP, U20 FDG6323L-TP, U21 FDG6323L-TP, U22 FDG6323L-TP, U23 FDG6323L-TP, U24 FDG6323L-TP, U7 FDG6323L-TP, U8 74LS596, U9 74LS596

Commit message: update
break down schemantic to panels, added controller and additional commponents, fixed
Parts:
- added J8: Conn_01x08, Connector_PinSocket_2.54mm:PinSocket_1x08_P2.54mm_Vertical, symbol Connector_Generic:Conn_01x08
Connections:
- net A_IN: now also J8.5 (Pin_5)
- net GND: now also J8.7 (Pin_7)
- net RCLK_A: now also J8.3 (Pin_3)
- net SRCLK_A: now also J8.2 (Pin_2)
- net V_LED: now also J8.8 (Pin_8)
- net _SRCLR_A: now also J8.1 (Pin_1)
- net +3.3V renamed +3V3
- net +3V3: now also J8.6 (Pin_6)
- no-connect marks 0 -> 1
